Commit message: done!

File: lite6_description/drake_urdf/gripper/lite6_normal_parallel_gripper.urdf (robot description, URDF)
Before this commit: robot lite6_normal_parallel_gripper, 4 links, 3 joints
Links:
- removed link link_tcp
- added link link_eef_tip
Joints:
- removed joint joint_tcp
- added joint joint_eef_tip: type fixed, parent lite6_normal_parallel_gripper_link, child link_eef_tip, origin xyz=0 0 0.0836 rpy=0 0 0

File: lite6_description/drake_urdf/gripper/lite6_reverse_parallel_gripper.urdf (robot description, URDF)
Before this commit: robot lite6_reverse_parallel_gripper, 4 links, 3 joints
Links:
- removed link link_tcp
- added link link_eef_tip
Joints:
- removed joint joint_tcp
- added joint joint_eef_tip: type fixed, parent lite6_reverse_parallel_gripper_link, child link_eef_tip, origin xyz=0 0 0.0836 rpy=0 0 0

File: lite6_description/drake_urdf/gripper/lite6_vacuum_gripper.urdf (robot description, URDF)
Before this commit: robot lite6_vacuum_gripper, 2 links, 1 joints
Links:
- removed link link_tcp
- added link link_eef_tip
Joints:
- removed joint joint_tcp
- added joint joint_eef_tip: type fixed, parent lite6_vacuum_gripper_link, child link_eef_tip, origin xyz=0 0 0.061 rpy=0 0 0

File: lite6_description/drake_urdf/robot_with_gripper/lite6_robot_with_normal_parallel_gripper.urdf (robot description, URDF)
Before this commit: robot lite6_robot_with_normal_parallel_gripper, 12 links, 11 joints
Links:
- removed link link_eef
- removed link link_tcp
- added link link_eef_tip
Joints:
- removed joint gripper_fix
- removed joint joint_eef
- removed joint joint_tcp
- removed joint left_parallel_gripper_joint
- removed joint right_parallel_gripper_joint
- added joint joint_eef_tip: type fixed, parent lite6_normal_parallel_gripper_link, child link_eef_tip, origin xyz=0 0 0.0836 rpy=0 0 0
- added joint joint_gripper_connector: type fixed, parent link6, child lite6_normal_parallel_gripper_link, origin xyz=0 0 0 rpy=0 0 0
- added joint joint_left_parallel_gripper: type prismatic, parent lite6_normal_parallel_gripper_link, child left_parallel_gripper, origin xyz=0 0.0025 0.0586 rpy=0 0 0, axis 0 1 0, limit lower=0 upper=0.008 effort=100.0 velocity=0.01
- added joint joint_right_parallel_gripper: type prismatic, parent lite6_normal_parallel_gripper_link, child right_parallel_gripper, origin xyz=0 -0.0025 0.0586 rpy=0 0 0, axis 0 1 0, limit lower=-0.008 upper=0. effort=100.0 velocity=0.01

File: lite6_description/drake_urdf/robot_with_gripper/lite6_robot_with_reverse_parallel_gripper.urdf (robot description, URDF)
Before this commit: robot lite6_robot_with_reverse_parallel_gripper, 12 links, 11 joints
Links:
- removed link link_eef
- removed link link_tcp
- added link link_eef_tip
Joints:
- removed joint gripper_fix
- removed joint joint_eef
- removed joint joint_tcp
- removed joint left_parallel_gripper_joint
- removed joint right_parallel_gripper_joint
- added joint joint_eef_tip: type fixed, parent lite6_reverse_parallel_gripper_link, child link_eef_tip, origin xyz=0 0 0.0836 rpy=0 0 0
- added joint joint_gripper_connector: type fixed, parent link6, child lite6_reverse_parallel_gripper_link, origin xyz=0 0 0 rpy=0 0 0
- added joint joint_left_parallel_gripper: type prismatic, parent lite6_reverse_parallel_gripper_link, child left_parallel_gripper, origin xyz=0 0.0135 0.0586 rpy=0 0 0, axis 0 1 0, limit lower=0 upper=0.008 effort=100.0 velocity=0.01
- added joint joint_right_parallel_gripper: type prismatic, parent lite6_reverse_parallel_gripper_link, child right_parallel_gripper, origin xyz=0 -0.0135 0.0586 rpy=0 0 0, axis 0 1 0, limit lower=-0.008 upper=0. effort=100.0 velocity=0.01

File: lite6_description/drake_urdf/robot_with_gripper/lite6_robot_with_vacuum_gripper.urdf (robot description, URDF)
Before this commit: robot lite6_robot_with_vacuum_gripper, 10 links, 9 joints
Links:
- removed link link_eef
- removed link link_tcp
- added link link_eef_tip
Joints:
- removed joint gripper_fix
- removed joint joint_eef
- removed joint joint_tcp
- added joint joint_eef_tip: type fixed, parent lite6_vacuum_gripper_link, child link_eef_tip, origin xyz=0 0 0.061 rpy=0 0 0
- added joint joint_gripper_connector: type fixed, parent link6, child lite6_vacuum_gripper_link, origin xyz=0 0 0 rpy=0 0 0

File: lite6_description/urdf/gripper/lite6_normal_parallel_gripper.urdf (robot description, URDF)
Before this commit: robot lite6_normal_parallel_gripper, 4 links, 3 joints
Links:
- removed link link_tcp
- added link link_eef_tip
Joints:
- removed joint joint_tcp
- added joint joint_eef_tip: type fixed, parent lite6_normal_parallel_gripper_link, child link_eef_tip, origin xyz=0 0 0.0836 rpy=0 0 0

File: lite6_description/urdf/gripper/lite6_reverse_parallel_gripper.urdf (robot description, URDF)
Before this commit: robot lite6_reverse_parallel_gripper, 4 links, 3 joints
Links:
- removed link link_tcp
- added link link_eef_tip
Joints:
- removed joint joint_tcp
- added joint joint_eef_tip: type fixed, parent lite6_reverse_parallel_gripper_link, child link_eef_tip, origin xyz=0 0 0.0836 rpy=0 0 0

File: lite6_description/urdf/gripper/lite6_vacuum_gripper.urdf (robot description, URDF)
Before this commit: robot lite6_vacuum_gripper, 2 links, 1 joints
Links:
- removed link link_tcp
- added link link_eef_tip
Joints:
- removed joint joint_tcp
- added joint joint_eef_tip: type fixed, parent lite6_vacuum_gripper_link, child link_eef_tip, origin xyz=0 0 0.061 rpy=0 0 0

File: lite6_description/urdf/robot_with_gripper/lite6_robot_with_normal_parallel_gripper.urdf (robot description, URDF)
Before this commit: robot lite6_robot_with_normal_parallel_gripper, 12 links, 11 joints
Links:
- removed link link_eef
- removed link link_tcp
- added link link_eef_tip
Joints:
- removed joint gripper_fix
- removed joint joint_eef
- removed joint joint_tcp
- removed joint left_parallel_gripper_joint
- removed joint right_parallel_gripper_joint
- added joint joint_eef_tip: type fixed, parent lite6_normal_parallel_gripper_link, child link_eef_tip, origin xyz=0 0 0.0836 rpy=0 0 0
- added joint joint_gripper_connector: type fixed, parent link6, child lite6_normal_parallel_gripper_link, origin xyz=0 0 0 rpy=0 0 0
- added joint joint_left_parallel_gripper: type prismatic, parent lite6_normal_parallel_gripper_link, child left_parallel_gripper, origin xyz=0 0.0025 0.0586 rpy=0 0 0, axis 0 1 0, limit lower=0 upper=0.008 effort=100.0 velocity=0.01
- added joint joint_right_parallel_gripper: type prismatic, parent lite6_normal_parallel_gripper_link, child right_parallel_gripper, origin xyz=0 -0.0025 0.0586 rpy=0 0 0, axis 0 1 0, limit lower=-0.008 upper=0. effort=100.0 velocity=0.01

File: lite6_description/urdf/robot_with_gripper/lite6_robot_with_reverse_parallel_gripper.urdf (robot description, URDF)
Before this commit: robot lite6_robot_with_reverse_parallel_gripper, 12 links, 11 joints
Links:
- removed link link_eef
- removed link link_tcp
- added link link_eef_tip
Joints:
- removed joint gripper_fix
- removed joint joint_eef
- removed joint joint_tcp
- added joint joint_eef_tip: type fixed, parent lite6_reverse_parallel_gripper_link, child link_eef_tip, origin xyz=0 0 0.0836 rpy=0 0 0
- added joint joint_gripper_connector: type fixed, parent link6, child lite6_reverse_parallel_gripper_link, origin xyz=0 0 0 rpy=0 0 0

File: lite6_description/urdf/robot_with_gripper/lite6_robot_with_vacuum_gripper.urdf (robot description, URDF)
Before this commit: robot lite6_robot_with_vacuum_gripper, 10 links, 9 joints
Links:
- removed link link_eef
- removed link link_tcp
- added link link_eef_tip
Joints:
- removed joint gripper_fix
- removed joint joint_eef
- removed joint joint_tcp
- added joint joint_eef_tip: type fixed, parent lite6_vacuum_gripper_link, child link_eef_tip, origin xyz=0 0 0.061 rpy=0 0 0
- added joint joint_gripper_connector: type fixed, parent link6, child lite6_vacuum_gripper_link, origin xyz=0 0 0 rpy=0 0 0

Commit message: fix gripper collision + inertias

File: lite6_description/drake_urdf/gripper/lite6_normal_parallel_gripper.urdf (robot description, URDF)
Before this commit: robot lite6_normal_parallel_gripper, 4 links, 3 joints
Links:
- link left_parallel_gripper: mass None -> 0.005; geometry collision box size=0.02 0.005 0.025; visual box size=0.02 0.005 0.025
- link right_parallel_gripper: mass None -> 0.005; geometry collision box size=0.02 0.005 0.025; visual box size=0.02 0.005 0.025

File: lite6_description/drake_urdf/gripper/lite6_reverse_parallel_gripper.urdf (robot description, URDF)
Before this commit: robot lite6_reverse_parallel_gripper, 4 links, 3 joints
Links:
- link left_parallel_gripper: mass None -> 0.005; geometry collision box size=0.02 0.005 0.025; visual box size=0.02 0.005 0.025
- link right_parallel_gripper: mass None -> 0.005; geometry collision box size=0.02 0.005 0.025; visual box size=0.02 0.005 0.025

File: lite6_description/drake_urdf/robot_with_gripper/lite6_robot_with_normal_parallel_gripper.urdf (robot description, URDF)
Before this commit: robot lite6_robot_with_normal_parallel_gripper, 11 links, 10 joints
Links:
- link left_parallel_gripper: mass None -> 0.005; geometry collision box size=0.02 0.005 0.025; visual box size=0.02 0.005 0.025
- link right_parallel_gripper: mass None -> 0.005; geometry collision box size=0.02 0.005 0.025; visual box size=0.02 0.005 0.025

File: lite6_description/drake_urdf/robot_with_gripper/lite6_robot_with_reverse_parallel_gripper.urdf (robot description, URDF)
Before this commit: robot lite6_robot_with_reverse_parallel_gripper, 11 links, 10 joints
Links:
- link left_parallel_gripper: mass None -> 0.005; geometry collision box size=0.02 0.005 0.025; visual box size=0.02 0.005 0.025
- link right_parallel_gripper: mass None -> 0.005; geometry collision box size=0.02 0.005 0.025; visual box size=0.02 0.005 0.025

File: lite6_description/urdf/gripper/lite6_normal_parallel_gripper.urdf (robot description, URDF)
Before this commit: robot lite6_normal_parallel_gripper, 4 links, 3 joints
Links:
- link left_parallel_gripper: mass None -> 0.005; geometry collision box size=0.02 0.005 0.025; visual box size=0.02 0.005 0.025
- link right_parallel_gripper: mass None -> 0.005; geometry collision box size=0.02 0.005 0.025; visual box size=0.02 0.005 0.025

File: lite6_description/urdf/gripper/lite6_reverse_parallel_gripper.urdf (robot description, URDF)
Before this commit: robot lite6_reverse_parallel_gripper, 4 links, 3 joints
Links:
- link left_parallel_gripper: mass None -> 0.005; geometry collision box size=0.02 0.005 0.025; visual box size=0.02 0.005 0.025
- link right_parallel_gripper: mass None -> 0.005; geometry collision box size=0.02 0.005 0.025; visual box size=0.02 0.005 0.025

File: lite6_description/urdf/robot_with_gripper/lite6_robot_with_normal_parallel_gripper.urdf (robot description, URDF)
Before this commit: robot lite6_robot_with_normal_parallel_gripper, 11 links, 10 joints
Links:
- link left_parallel_gripper: mass None -> 0.005; geometry collision box size=0.02 0.005 0.025; visual box size=0.02 0.005 0.025
- link right_parallel_gripper: mass None -> 0.005; geometry collision box size=0.02 0.005 0.025; visual box size=0.02 0.005 0.025

File: lite6_description/urdf/robot_with_gripper/lite6_robot_with_reverse_parallel_gripper.urdf (robot description, URDF)
Before this commit: robot lite6_robot_with_reverse_parallel_gripper, 11 links, 10 joints
Links:
- link left_parallel_gripper: mass None -> 0.005; geometry collision box size=0.02 0.005 0.025; visual box size=0.02 0.005 0.025
- link right_parallel_gripper: mass None -> 0.005; geometry collision box size=0.02 0.005 0.025; visual box size=0.02 0.005 0.025
