Commit message: fix

File: lite6_description/drake_urdf/robot_with_gripper/lite6_robot_with_unactuated_normal_parallel_gripper.urdf (robot description, URDF)
Before this commit: robot lite6_robot_with_unactuated_normal_parallel_gripper, 11 links, 8 joints
Joints:
- added joint joint_left_parallel_gripper: type fixed, parent lite6_normal_parallel_gripper_link, child left_parallel_gripper_link, origin xyz=0 0.0025 0.0586 rpy=0 0 0
- added joint joint_right_parallel_gripper: type fixed, parent lite6_normal_parallel_gripper_link, child right_parallel_gripper_link, origin xyz=0 -0.0025 0.0586 rpy=0 0 0

File: lite6_description/drake_urdf/robot_with_gripper/lite6_robot_with_unactuated_reverse_parallel_gripper.urdf (robot description, URDF)
Before this commit: robot lite6_robot_with_unactuated_reverse_parallel_gripper, 11 links, 8 joints
Joints:
- added joint joint_left_parallel_gripper: type fixed, parent lite6_reverse_parallel_gripper_link, child left_parallel_gripper_link, origin xyz=0 0.0135 0.0586 rpy=0 0 0
- added joint joint_right_parallel_gripper: type fixed, parent lite6_reverse_parallel_gripper_link, child right_parallel_gripper_link, origin xyz=0 -0.0135 0.0586 rpy=0 0 0

File: lite6_description/urdf/robot_with_gripper/lite6_robot_with_unactuated_normal_parallel_gripper.urdf (robot description, URDF)
Before this commit: robot lite6_robot_with_unactuated_normal_parallel_gripper, 11 links, 8 joints
Joints:
- added joint joint_left_parallel_gripper: type fixed, parent lite6_normal_parallel_gripper_link, child left_parallel_gripper_link, origin xyz=0 0.0025 0.0586 rpy=0 0 0
- added joint joint_right_parallel_gripper: type fixed, parent lite6_normal_parallel_gripper_link, child right_parallel_gripper_link, origin xyz=0 -0.0025 0.0586 rpy=0 0 0

File: lite6_description/urdf/robot_with_gripper/lite6_robot_with_unactuated_reverse_parallel_gripper.urdf (robot description, URDF)
Before this commit: robot lite6_robot_with_unactuated_reverse_parallel_gripper, 11 links, 10 joints
Joints:
- joint left_parallel_gripper_joint: axis 0 1 0 -> (none); limit lower=0 upper=0.008 effort=100.0 velocity=0.01 -> (none); type prismatic -> fixed
- joint right_parallel_gripper_joint: axis 0 1 0 -> (none); limit lower=-0.008 upper=0. effort=100.0 velocity=0.01 -> (none); type prismatic -> fixed
