Commit message: update

File: lite6_description/drake_urdf/robot_with_gripper/lite6_robot_with_actuated_normal_parallel_gripper.urdf (robot description, URDF)
Before this commit: robot lite6_robot_without_gripper, 8 links, 7 joints
Links:
- removed link link_eef
- added link left_parallel_gripper_link, mass 0.005; collision box size=0.02 0.005 0.025; visual box size=0.02 0.005 0.025
- added link link_eef_tip
- added link lite6_normal_parallel_gripper_link, mass 0.28; collision mesh filename=package://lite6_description/meshes/gripper/collision/parall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; collision mesh filename=package://lite6_description/meshes/gripper/collision/parall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
- added link right_parallel_gripper_link, mass 0.005; collision box size=0.02 0.005 0.025; visual box size=0.02 0.005 0.025
Joints:
- removed joint joint_eef
- added joint joint_eef_tip: type fixed, parent lite6_normal_parallel_gripper_link, child link_eef_tip, origin xyz=0 0 0.0836 rpy=0 0 0
- added joint joint_gripper_connector: type fixed, parent link6, child lite6_normal_parallel_gripper_link, origin xyz=0 0 0 rpy=0 0 0
- added joint joint_left_parallel_gripper: type prismatic, parent lite6_normal_parallel_gripper_link, child left_parallel_gripper_link, origin xyz=0 0.0025 0.0586 rpy=0 0 0, axis 0 1 0, limit lower=0 upper=0.008 effort=100.0 velocity=0.01
- added joint joint_right_parallel_gripper: type prismatic, parent lite6_normal_parallel_gripper_link, child right_parallel_gripper_link, origin xyz=0 -0.0025 0.0586 rpy=0 0 0, axis 0 1 0, limit lower=-0.008 upper=0. effort=100.0 velocity=0.01

File: lite6_description/drake_urdf/robot_with_gripper/lite6_robot_with_actuated_reverse_parallel_gripper.urdf (robot description, URDF)
Before this commit: robot lite6_robot_with_reverse_parallel_gripper, 11 links, 10 joints
Links:
- removed link left_parallel_gripper
- removed link right_parallel_gripper
- added link left_parallel_gripper_link, mass 0.005; collision box size=0.02 0.005 0.025; visual box size=0.02 0.005 0.025
- added link right_parallel_gripper_link, mass 0.005; collision box size=0.02 0.005 0.025; visual box size=0.02 0.005 0.025
Joints:
- removed joint left_parallel_gripper_joint
- removed joint right_parallel_gripper_joint
- added joint joint_left_parallel_gripper: type prismatic, parent lite6_reverse_parallel_gripper_link, child left_parallel_gripper_link, origin xyz=0 0.0135 0.0586 rpy=0 0 0, axis 0 1 0, limit lower=0 upper=0.008 effort=100.0 velocity=0.01
- added joint joint_right_parallel_gripper: type prismatic, parent lite6_reverse_parallel_gripper_link, child right_parallel_gripper_link, origin xyz=0 -0.0135 0.0586 rpy=0 0 0, axis 0 1 0, limit lower=-0.008 upper=0. effort=100.0 velocity=0.01

File: lite6_description/drake_urdf/robot_with_gripper/lite6_robot_with_unactuated_normal_parallel_gripper.urdf (robot description, URDF)
Before this commit: robot lite6_robot_without_gripper, 8 links, 7 joints
Links:
- removed link link_eef
- added link left_parallel_gripper_link, mass 0.005; collision box size=0.02 0.005 0.025; visual box size=0.02 0.005 0.025
- added link link_eef_tip
- added link lite6_normal_parallel_gripper_link, mass 0.28; collision mesh filename=package://lite6_description/meshes/gripper/collision/parall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; collision mesh filename=package://lite6_description/meshes/gripper/collision/parall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
- added link right_parallel_gripper_link, mass 0.005; collision box size=0.02 0.005 0.025; visual box size=0.02 0.005 0.025
Joints:
- removed joint joint_eef
- added joint joint_eef_tip: type fixed, parent lite6_normal_parallel_gripper_link, child link_eef_tip, origin xyz=0 0 0.0836 rpy=0 0 0
- added joint joint_gripper_connector: type fixed, parent link6, child lite6_normal_parallel_gripper_link, origin xyz=0 0 0 rpy=0 0 0

File: lite6_description/drake_urdf/robot_with_gripper/lite6_robot_with_unactuated_reverse_parallel_gripper.urdf (robot description, URDF)
Before this commit: robot lite6_robot_with_normal_parallel_gripper, 11 links, 10 joints
Links:
- removed link left_parallel_gripper
- removed link lite6_normal_parallel_gripper_link
- removed link right_parallel_gripper
- added link left_parallel_gripper_link, mass 0.005; collision box size=0.02 0.005 0.025; visual box size=0.02 0.005 0.025
- added link lite6_reverse_parallel_gripper_link, mass 0.28; collision mesh filename=package://lite6_description/meshes/gripper/collision/parall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; collision mesh filename=package://lite6_description/meshes/gripper/collision/parall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
- added link right_parallel_gripper_link, mass 0.005; collision box size=0.02 0.005 0.025; visual box size=0.02 0.005 0.025
Joints:
- removed joint joint_left_parallel_gripper
- removed joint joint_right_parallel_gripper
- joint joint_eef_tip: parent lite6_normal_parallel_gripper_link -> lite6_reverse_parallel_gripper_link
- joint joint_gripper_connector: child lite6_normal_parallel_gripper_link -> lite6_reverse_parallel_gripper_link

File: lite6_description/urdf/robot_with_gripper/lite6_robot_with_actuated_normal_parallel_gripper.urdf (robot description, URDF)
Before this commit: robot lite6_robot_without_gripper, 8 links, 7 joints
Links:
- removed link link_eef
- added link left_parallel_gripper_link, mass 0.005; collision box size=0.02 0.005 0.025; visual box size=0.02 0.005 0.025
- added link link_eef_tip
- added link lite6_normal_parallel_gripper_link, mass 0.28; collision mesh filename=package://lite6_description/meshes/gripper/collision/parall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; collision mesh filename=package://lite6_description/meshes/gripper/collision/parall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
- added link right_parallel_gripper_link, mass 0.005; collision box size=0.02 0.005 0.025; visual box size=0.02 0.005 0.025
Joints:
- removed joint joint_eef
- added joint joint_eef_tip: type fixed, parent lite6_normal_parallel_gripper_link, child link_eef_tip, origin xyz=0 0 0.0836 rpy=0 0 0
- added joint joint_gripper_connector: type fixed, parent link6, child lite6_normal_parallel_gripper_link, origin xyz=0 0 0 rpy=0 0 0
- added joint joint_left_parallel_gripper: type prismatic, parent lite6_normal_parallel_gripper_link, child left_parallel_gripper_link, origin xyz=0 0.0025 0.0586 rpy=0 0 0, axis 0 1 0, limit lower=0 upper=0.008 effort=100.0 velocity=0.01
- added joint joint_right_parallel_gripper: type prismatic, parent lite6_normal_parallel_gripper_link, child right_parallel_gripper_link, origin xyz=0 -0.0025 0.0586 rpy=0 0 0, axis 0 1 0, limit lower=-0.008 upper=0. effort=100.0 velocity=0.01

File: lite6_description/urdf/robot_with_gripper/lite6_robot_with_actuated_reverse_parallel_gripper.urdf (robot description, URDF)
Before this commit: robot lite6_robot_with_reverse_parallel_gripper, 11 links, 10 joints
Links:
- removed link left_parallel_gripper
- removed link right_parallel_gripper
- added link left_parallel_gripper_link, mass 0.005; collision box size=0.02 0.005 0.025; visual box size=0.02 0.005 0.025
- added link right_parallel_gripper_link, mass 0.005; collision box size=0.02 0.005 0.025; visual box size=0.02 0.005 0.025
Joints:
- removed joint joint_left_parallel_gripper
- removed joint joint_right_parallel_gripper
- added joint left_parallel_gripper_joint: type prismatic, parent lite6_reverse_parallel_gripper_link, child left_parallel_gripper_link, origin xyz=0 0.0135 0.0586 rpy=0 0 0, axis 0 1 0, limit lower=0 upper=0.008 effort=100.0 velocity=0.01
- added joint right_parallel_gripper_joint: type prismatic, parent lite6_reverse_parallel_gripper_link, child right_parallel_gripper_link, origin xyz=0 -0.0135 0.0586 rpy=0 0 0, axis 0 1 0, limit lower=-0.008 upper=0. effort=100.0 velocity=0.01

File: lite6_description/urdf/robot_with_gripper/lite6_robot_with_unactuated_normal_parallel_gripper.urdf (robot description, URDF)
Before this commit: robot lite6_robot_with_normal_parallel_gripper, 11 links, 10 joints
Links:
- removed link left_parallel_gripper
- removed link right_parallel_gripper
- added link left_parallel_gripper_link, mass 0.005; collision box size=0.02 0.005 0.025; visual box size=0.02 0.005 0.025
- added link right_parallel_gripper_link, mass 0.005; collision box size=0.02 0.005 0.025; visual box size=0.02 0.005 0.025
Joints:
- removed joint joint_left_parallel_gripper
- removed joint joint_right_parallel_gripper

File: lite6_description/urdf/robot_with_gripper/lite6_robot_with_unactuated_reverse_parallel_gripper.urdf (robot description, URDF)
Before this commit: robot lite6_robot_without_gripper, 8 links, 7 joints
Links:
- removed link link_eef
- added link left_parallel_gripper_link, mass 0.005; collision box size=0.02 0.005 0.025; visual box size=0.02 0.005 0.025
- added link link_eef_tip
- added link lite6_reverse_parallel_gripper_link, mass 0.28; collision mesh filename=package://lite6_description/meshes/gripper/collision/parall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; collision mesh filename=package://lite6_description/meshes/gripper/collision/parall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
- added link right_parallel_gripper_link, mass 0.005; collision box size=0.02 0.005 0.025; visual box size=0.02 0.005 0.025
Joints:
- removed joint joint_eef
- added joint joint_eef_tip: type fixed, parent lite6_reverse_parallel_gripper_link, child link_eef_tip, origin xyz=0 0 0.0836 rpy=0 0 0
- added joint joint_gripper_connector: type fixed, parent link6, child lite6_reverse_parallel_gripper_link, origin xyz=0 0 0 rpy=0 0 0
- added joint left_parallel_gripper_joint: type prismatic, parent lite6_reverse_parallel_gripper_link, child left_parallel_gripper_link, origin xyz=0 0.0135 0.0586 rpy=0 0 0, axis 0 1 0, limit lower=0 upper=0.008 effort=100.0 velocity=0.01
- added joint right_parallel_gripper_joint: type prismatic, parent lite6_reverse_parallel_gripper_link, child right_parallel_gripper_link, origin xyz=0 -0.0135 0.0586 rpy=0 0 0, axis 0 1 0, limit lower=-0.008 upper=0. effort=100.0 velocity=0.01

Commit message: change

File: lite6_description/drake_urdf/robot_with_gripper/lite6_robot_with_actuated_normal_parallel_gripper.urdf (robot description, URDF)
Before this commit: robot lite6_robot_with_actuated_normal_parallel_gripper, 11 links, 10 joints
Joints:
- joint joint_left_parallel_gripper: limit lower=0 upper=0.008 effort=100.0 velocity=0.01 -> lower=0 upper=0.008 effort=100.0 velocity=0.1
- joint joint_right_parallel_gripper: limit lower=-0.008 upper=0. effort=100.0 velocity=0.01 -> lower=-0.008 upper=0. effort=100.0 velocity=0.1

File: lite6_description/drake_urdf/robot_with_gripper/lite6_robot_with_actuated_reverse_parallel_gripper.urdf (robot description, URDF)
Before this commit: robot lite6_robot_with_actuated_reverse_parallel_gripper, 11 links, 10 joints
Joints:
- joint joint_left_parallel_gripper: limit lower=0 upper=0.008 effort=100.0 velocity=0.01 -> lower=0 upper=0.008 effort=100.0 velocity=0.1
- joint joint_right_parallel_gripper: limit lower=-0.008 upper=0. effort=100.0 velocity=0.01 -> lower=-0.008 upper=0. effort=100.0 velocity=0.1

File: lite6_description/urdf/robot_with_gripper/lite6_robot_with_actuated_normal_parallel_gripper.urdf (robot description, URDF)
Before this commit: robot lite6_robot_with_actuated_normal_parallel_gripper, 11 links, 10 joints
Joints:
- joint joint_left_parallel_gripper: limit lower=0 upper=0.008 effort=100.0 velocity=0.01 -> lower=0 upper=0.008 effort=100.0 velocity=0.1
- joint joint_right_parallel_gripper: limit lower=-0.008 upper=0. effort=100.0 velocity=0.01 -> lower=-0.008 upper=0. effort=100.0 velocity=0.1

File: lite6_description/urdf/robot_with_gripper/lite6_robot_with_actuated_reverse_parallel_gripper.urdf (robot description, URDF)
Before this commit: robot lite6_robot_with_actuated_reverse_parallel_gripper, 11 links, 10 joints
Joints:
- joint left_parallel_gripper_joint: limit lower=0 upper=0.008 effort=100.0 velocity=0.01 -> lower=0 upper=0.008 effort=100.0 velocity=0.1
- joint right_parallel_gripper_joint: limit lower=-0.008 upper=0. effort=100.0 velocity=0.01 -> lower=-0.008 upper=0. effort=100.0 velocity=0.1
