Commit message: mostly done. Actuators left

File: h1_description/drake_urdf/h1.urdf (robot description, URDF)
Before this commit: robot h1_description, 22 links, 21 joints
Links:
- link left_elbow_link: geometry collision cylinder length=0.28 radius=0.03; visual mesh filename=package://h1_description/meshes/left_elbow_link.dae
- link left_hip_yaw_link: geometry collision cylinder length=0.08 radius=0.05; visual mesh filename=package://h1_description/meshes/left_hip_yaw_link.dae
- link left_shoulder_pitch_link: geometry collision cylinder length=0.06 radius=0.05; visual mesh filename=package://h1_description/meshes/left_shoulder_pitch_link.dae
- link left_shoulder_roll_link: geometry collision cylinder length=0.08 radius=0.04; collision cylinder length=0.08 radius=0.05
- link left_shoulder_yaw_link: geometry collision cylinder length=0.15 radius=0.03; visual mesh filename=package://h1_description/meshes/left_shoulder_yaw_link.dae
- link right_elbow_link: geometry collision cylinder length=0.28 radius=0.03; visual mesh filename=package://h1_description/meshes/right_elbow_link.dae
- link right_hip_yaw_link: geometry collision cylinder length=0.08 radius=0.05; visual mesh filename=package://h1_description/meshes/right_hip_yaw_link.dae
- link right_shoulder_pitch_link: geometry collision cylinder length=0.06 radius=0.05; visual mesh filename=package://h1_description/meshes/right_shoulder_pitch_link.d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
- link right_shoulder_roll_link: geometry collision cylinder length=0.08 radius=0.04; collision cylinder length=0.08 radius=0.05
- link right_shoulder_yaw_link: geometry collision cylinder length=0.15 radius=0.03; visual mesh filename=package://h1_description/meshes/right_shoulder_yaw_link.dae
- link torso_link: geometry collision box size=0.14 0.20 0.45; collision sphere radius=0.08
