Commit message: done?

File: h1_description/urdf/h1.urdf (robot description, URDF)
Before this commit: robot h1_description, 22 links, 21 joints
Links:
- link left_ankle_link: geometry collision box size=0.30 0.03 0.024; visual mesh filename=package://h1_description/meshes/left_ankle_link.dae
- link left_elbow_link: geometry collision cylinder length=0.28 radius=0.03; visual mesh filename=package://h1_description/meshes/left_elbow_link.dae
- link left_hip_pitch_link: geometry collision box size=0.05 0.05 0.34; collision cylinder length=0.1 radius=0.065
- link left_hip_roll_link: geometry collision cylinder length=0.19 radius=0.06; visual mesh filename=package://h1_description/meshes/left_hip_roll_link.dae
- link left_hip_yaw_link: geometry collision cylinder length=0.08 radius=0.05; visual mesh filename=package://h1_description/meshes/left_hip_yaw_link.dae
- link left_knee_link: geometry collision box size=0.05 0.05 0.35; visual mesh filename=package://h1_description/meshes/left_knee_link.dae
- link left_shoulder_pitch_link: geometry collision cylinder length=0.06 radius=0.05; visual mesh filename=package://h1_description/meshes/left_shoulder_pitch_link.dae
- link left_shoulder_roll_link: geometry collision cylinder length=0.08 radius=0.04; collision cylinder length=0.08 radius=0.05
- link left_shoulder_yaw_link: geometry collision cylinder length=0.15 radius=0.03; visual mesh filename=package://h1_description/meshes/left_shoulder_yaw_link.dae
- link pelvis: geometry collision box size=0.14 0.1 0.08; visual mesh filename=package://h1_description/meshes/pelvis.dae
- link right_ankle_link: geometry collision box size=0.30 0.03 0.024; visual mesh filename=package://h1_description/meshes/right_ankle_link.dae
- link right_elbow_link: geometry collision cylinder length=0.28 radius=0.03; visual mesh filename=package://h1_description/meshes/right_elbow_link.dae
- link right_hip_pitch_link: geometry collision box size=0.05 0.05 0.34; collision cylinder length=0.1 radius=0.065
- link right_hip_roll_link: geometry collision cylinder length=0.19 radius=0.06; visual mesh filename=package://h1_description/meshes/right_hip_roll_link.dae
- link right_hip_yaw_link: geometry collision cylinder length=0.08 radius=0.05; visual mesh filename=package://h1_description/meshes/right_hip_yaw_link.dae
- link right_knee_link: geometry collision box size=0.05 0.05 0.35; visual mesh filename=package://h1_description/meshes/right_knee_link.dae
- link right_shoulder_pitch_link: geometry collision cylinder length=0.06 radius=0.05; visual mesh filename=package://h1_description/meshes/right_shoulder_pitch_link.d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
- link right_shoulder_roll_link: geometry collision cylinder length=0.08 radius=0.04; collision cylinder length=0.08 radius=0.05
- link right_shoulder_yaw_link: geometry collision cylinder length=0.15 radius=0.03; visual mesh filename=package://h1_description/meshes/right_shoulder_yaw_link.dae
- link torso_link: geometry collision box size=0.14 0.20 0.45; collision sphere radius=0.08
