Commit message: for gravity comp

File: rebot_b601_dm_description/drake_urdf/rebot_b601_dm_with_gripper.urdf (robot description, URDF)
Before this commit: robot rebot_b601_dm_with_gripper, 11 links, 10 joints
Links:
- link base_link: mass 0.79874480798149 -> 0.83660000
- link gripper_link: mass 0.181800159145243 -> 0.36534420980225685
- link link1: mass 0.0840736498625263 -> 0.16130000
- link link2: mass 0.710394385134637 -> 1.32660000
- link link3: mass 0.524941641478664 -> 0.83530000
- link link4: mass 0.191139210973019 -> 0.52000000
- link link5: mass 0.150004102113546 -> 0.38300000
- link link6: mass 0.0187271664583674 -> 0.36630000

File: rebot_b601_dm_description/urdf/rebot_b601_dm_with_gripper.urdf (robot description, URDF)
Before this commit: robot rebot_b601_dm_with_gripper, 11 links, 10 joints
Links:
- link base_link: mass 0.79874480798149 -> 0.83660000
- link gripper_link: mass 0.181800159145243 -> 0.36534420980225685
- link link1: mass 0.0840736498625263 -> 0.16130000
- link link2: mass 0.710394385134637 -> 1.32660000
- link link3: mass 0.524941641478664 -> 0.83530000
- link link4: mass 0.191139210973019 -> 0.52000000
- link link5: mass 0.150004102113546 -> 0.38300000
- link link6: mass 0.0187271664583674 -> 0.36630000
